Commit message: kinda working example

File: rc_car_description/urdf/rc_car.xacro (robot description, xacro)
@@ -40,5 +40,5 @@
       <origin xyz="${chassis_x_offset} 0 0" rpy="0 0 0"/>
       <geometry>
-        <mesh filename="package://${pkg_name}/meshes/rc_car_chassis.stl" scale="1 1 1"/>
+        <mesh filename="file://$(find rc_car_description)/meshes/rc_car_chassis.stl" scale="1 1 1"/>
       </geometry>
       <material name="gray">
@@ -54,4 +54,15 @@
     <xacro:box_inertia m="1.5" w="0.12" h="0.05" d="0.25" x_offset="${chassis_x_offset}"/>
   </link>
+  <!-- Dummy Steering Wheel to satisfy the Ackermann plugin -->
+  <link name="steering_wheel_link">
+    <xacro:dummy_inertia/>
+  </link>
+  <joint name="steering_wheel_joint" type="revolute">
+    <parent link="base_link"/>
+    <child link="steering_wheel_link"/>
+    <origin xyz="0 0 0" rpy="0 0 0"/>
+    <axis xyz="0 0 1"/>
+    <limit lower="-${max_steer_angle}" upper="${max_steer_angle}" effort="10.0" velocity="10.0"/>
+  </joint>
   <xacro:macro name="rc_wheel" params="prefix mesh_rpy">
     <link name="${prefix}_wheel_link">
@@ -59,5 +70,5 @@
         <origin xyz="0 0 0" rpy="${mesh_rpy}"/>
         <geometry>
-          <mesh filename="package://${pkg_name}/meshes/rc_car_wheel.stl" scale="1 1 1"/>
+          <mesh filename="file://$(find rc_car_description)/meshes/rc_car_wheel.stl" scale="1 1 1"/>
         </geometry>
         <material name="black">
@@ -68,8 +79,8 @@
         <origin xyz="0 0 0" rpy="0 0 0"/>
         <geometry>
-          <sphere radius="${wheel_radius}"/>
+          <cylinder radius="${wheel_radius}" length="${wheel_width}"/>
         </geometry>
       </collision>
-      <xacro:cylinder_inertia m="0.1" r="${wheel_radius}" h="${wheel_width}"/>
+      <xacro:cylinder_inertia m="0.5" r="${wheel_radius}" h="${wheel_width}"/>
     </link>
     <gazebo reference="${prefix}_wheel_link">
@@ -88,6 +99,6 @@
     <origin xyz="0 ${track_width/2} 0" rpy="-${M_PI/2.0} 0 0"/>
     <axis xyz="0 0 1"/>
-    <limit effort="100.0" velocity="100.0"/>
-    </joint>
+    <limit effort="1.0" velocity="100.0"/>
+  </joint>
   <xacro:rc_wheel prefix="rear_right" mesh_rpy="${M_PI/2.0} 0 0"/>
   <joint name="rear_right_wheel_joint" type="continuous">
@@ -96,5 +107,5 @@
     <origin xyz="0 ${-track_width/2} 0" rpy="-${M_PI/2.0} 0 0"/>
     <axis xyz="0 0 1"/>
-    <limit effort="100.0" velocity="100.0"/>
+    <limit effort="1.0" velocity="100.0"/>
   </joint>
   <xacro:macro name="front_steer_assembly" params="prefix y_offset mesh_rpy">
@@ -115,5 +126,5 @@
       <origin xyz="0 0 0" rpy="-${M_PI/2.0} 0 0"/>
       <axis xyz="0 0 1"/>
-      <limit effort="100.0" velocity="100.0"/>
+      <limit effort="1.0" velocity="100.0"/>
     </joint>
   </xacro:macro>
@@ -126,4 +137,5 @@
         <remapping>cmd_vel:=cmd_vel</remapping>
         <remapping>odom:=odom</remapping>
+        <remapping>distance:=distance</remapping>
       </ros>
       <update_rate>100.0</update_rate>
@@ -134,7 +146,9 @@
       <left_steering_joint>front_left_steer_joint</left_steering_joint>
       <right_steering_joint>front_right_steer_joint</right_steering_joint>
+      <steering_wheel_joint>steering_wheel_joint</steering_wheel_joint>
       <wheel_separation>${track_width}</wheel_separation>
       <wheel_base>${wheelbase}</wheel_base>
       <steering_wheel_angle>${max_steer_angle}</steering_wheel_angle>
+      <wheel_radius>${wheel_radius}</wheel_radius>
       <max_steer>${max_steer_angle}</max_steer>
       <max_steering_angle>${max_steer_angle}</max_steering_angle>
@@ -142,7 +156,15 @@
       <odometry_frame>odom</odometry_frame>
       <robot_base_frame>base_footprint</robot_base_frame>
+      <!-- PID tuning -->
+      <left_steering_pid_gain>1.0 0.0 0.1</left_steering_pid_gain>
+      <left_steering_i_range>0 0</left_steering_i_range>
+      <right_steering_pid_gain>1.0 0.0 0.1</right_steering_pid_gain>
+      <right_steering_i_range>0 0</right_steering_i_range>
+      <linear_velocity_pid_gain>5.0 0.0 0.0</linear_velocity_pid_gain>
+      <linear_velocity_i_range>0 0</linear_velocity_i_range>
       <publish_odom>true</publish_odom>
       <publish_odom_tf>true</publish_odom_tf>
       <publish_wheel_tf>true</publish_wheel_tf>
+      <publish_distance>true</publish_distance>
     </plugin>
   </gazebo>

Commit message: first good working example

File: rc_car_description/urdf/rc_car.xacro (robot description, xacro)
@@ -100,4 +100,5 @@
     <axis xyz="0 0 1"/>
     <limit effort="1.0" velocity="100.0"/>
+    <dynamics damping="0.001" friction="0.001"/> <!-- Add this line -->
   </joint>
   <xacro:rc_wheel prefix="rear_right" mesh_rpy="${M_PI/2.0} 0 0"/>
@@ -108,4 +109,5 @@
     <axis xyz="0 0 1"/>
     <limit effort="1.0" velocity="100.0"/>
+    <dynamics damping="0.001" friction="0.001"/> <!-- Add this line -->
   </joint>
   <xacro:macro name="front_steer_assembly" params="prefix y_offset mesh_rpy">
@@ -119,4 +121,5 @@
       <axis xyz="0 0 1"/>
       <limit lower="-${max_steer_angle}" upper="${max_steer_angle}" effort="100.0" velocity="2.0"/>
+      <dynamics damping="0.001" friction="0.001"/> <!-- Add this line -->
     </joint>
     <xacro:rc_wheel prefix="${prefix}" mesh_rpy="${mesh_rpy}"/>
@@ -127,4 +130,5 @@
       <axis xyz="0 0 1"/>
       <limit effort="1.0" velocity="100.0"/>
+      <dynamics damping="0.001" friction="0.001"/> <!-- Add this line -->
     </joint>
   </xacro:macro>

Commit message: Changed the movement dynamics to reflect the real robot

File: rc_car_description/urdf/rc_car.xacro (robot description, xacro)
@@ -9,7 +9,7 @@
   <xacro:property name="max_steer_angle" value="0.523"/>
   <xacro:property name="M_PI" value="3.1415926535897931" />
-  <xacro:macro name="box_inertia" params="m w h d x_offset">
+  <xacro:macro name="box_inertia" params="m w h d x_offset z_offset">
     <inertial>
-      <origin xyz="${x_offset} 0 0" rpy="0 0 0"/>
+      <origin xyz="${x_offset} 0 ${z_offset}" rpy="0 0 0"/>
       <mass value="${m}"/>
       <inertia ixx="${(m/12) * (h*h + d*d)}" ixy="0.0" ixz="0.0" iyy="${(m/12) * (w*w + d*d)}" iyz="0.0" izz="${(m/12) * (w*w + h*h)}"/>
@@ -52,6 +52,5 @@
       </geometry>
     </collision>
-    <xacro:box_inertia m="1.5" w="0.12" h="0.05" d="0.25" x_offset="${chassis_x_offset}"/>
-  </link>
+<xacro:box_inertia m="1.5" w="0.12" h="0.05" d="0.25" x_offset="${chassis_x_offset}" z_offset="-0.02"/>  </link>
   <!-- Dummy Steering Wheel to satisfy the Ackermann plugin -->
   <link name="steering_wheel_link">
@@ -85,6 +84,6 @@
     </link>
     <gazebo reference="${prefix}_wheel_link">
-      <mu1>0.8</mu1>
-      <mu2>0.8</mu2>
+      <mu1>1.2</mu1>
+      <mu2>1.2</mu2>
       <kp>1000000.0</kp>
       <kd>100.0</kd>
@@ -99,6 +98,6 @@
     <origin xyz="0 ${track_width/2} 0" rpy="-${M_PI/2.0} 0 0"/>
     <axis xyz="0 0 1"/>
-    <limit effort="1.0" velocity="100.0"/>
-    <dynamics damping="0.001" friction="0.001"/> <!-- Add this line -->
+    <limit effort="5.0" velocity="100.0"/>
+    <dynamics damping="0.001" friction="0.05"/> <!-- Add this line -->
   </joint>
   <xacro:rc_wheel prefix="rear_right" mesh_rpy="${M_PI/2.0} 0 0"/>
@@ -108,6 +107,6 @@
     <origin xyz="0 ${-track_width/2} 0" rpy="-${M_PI/2.0} 0 0"/>
     <axis xyz="0 0 1"/>
-    <limit effort="1.0" velocity="100.0"/>
-    <dynamics damping="0.001" friction="0.001"/> <!-- Add this line -->
+    <limit effort="5.0" velocity="100.0"/>
+    <dynamics damping="0.001" friction="0.05"/> <!-- Add this line -->
   </joint>
   <xacro:macro name="front_steer_assembly" params="prefix y_offset mesh_rpy">
@@ -121,5 +120,5 @@
       <axis xyz="0 0 1"/>
       <limit lower="-${max_steer_angle}" upper="${max_steer_angle}" effort="100.0" velocity="2.0"/>
-      <dynamics damping="0.001" friction="0.001"/> <!-- Add this line -->
+      <dynamics damping="0.001" friction="0.05"/> <!-- Add this line -->
     </joint>
     <xacro:rc_wheel prefix="${prefix}" mesh_rpy="${mesh_rpy}"/>
@@ -129,6 +128,6 @@
       <origin xyz="0 0 0" rpy="-${M_PI/2.0} 0 0"/>
       <axis xyz="0 0 1"/>
-      <limit effort="1.0" velocity="100.0"/>
-      <dynamics damping="0.001" friction="0.001"/> <!-- Add this line -->
+      <limit effort="5.0" velocity="100.0"/>
+      <dynamics damping="0.001" friction="0.05"/> <!-- Add this line -->
     </joint>
   </xacro:macro>
@@ -157,11 +156,11 @@
       <max_steer>${max_steer_angle}</max_steer>
       <max_steering_angle>${max_steer_angle}</max_steering_angle>
-      <max_speed>2.0</max_speed>
+      <max_speed>5.0</max_speed>
       <odometry_frame>odom</odometry_frame>
       <robot_base_frame>base_footprint</robot_base_frame>
       <!-- PID tuning -->
-      <left_steering_pid_gain>1.0 0.0 0.1</left_steering_pid_gain>
+      <left_steering_pid_gain>10.0 0.0 0.1</left_steering_pid_gain>
       <left_steering_i_range>0 0</left_steering_i_range>
-      <right_steering_pid_gain>1.0 0.0 0.1</right_steering_pid_gain>
+      <right_steering_pid_gain>10.0 0.0 0.1</right_steering_pid_gain>
       <right_steering_i_range>0 0</right_steering_i_range>
       <linear_velocity_pid_gain>5.0 0.0 0.0</linear_velocity_pid_gain>

Commit message: added lidar, ultrasonic sensor and jetson model

File: rc_car_description/urdf/rc_car.xacro (robot description, xacro)
@@ -52,5 +52,6 @@
       </geometry>
     </collision>
-<xacro:box_inertia m="1.5" w="0.12" h="0.05" d="0.25" x_offset="${chassis_x_offset}" z_offset="-0.02"/>  </link>
+    <xacro:box_inertia m="1.5" w="0.12" h="0.05" d="0.25" x_offset="${chassis_x_offset}" z_offset="-0.02"/>
+  </link>
   <!-- Dummy Steering Wheel to satisfy the Ackermann plugin -->
   <link name="steering_wheel_link">
@@ -99,5 +100,5 @@
     <axis xyz="0 0 1"/>
     <limit effort="5.0" velocity="100.0"/>
-    <dynamics damping="0.001" friction="0.05"/> <!-- Add this line -->
+    <dynamics damping="0.001" friction="0.05"/>
   </joint>
   <xacro:rc_wheel prefix="rear_right" mesh_rpy="${M_PI/2.0} 0 0"/>
@@ -108,5 +109,5 @@
     <axis xyz="0 0 1"/>
     <limit effort="5.0" velocity="100.0"/>
-    <dynamics damping="0.001" friction="0.05"/> <!-- Add this line -->
+    <dynamics damping="0.001" friction="0.05"/>
   </joint>
   <xacro:macro name="front_steer_assembly" params="prefix y_offset mesh_rpy">
@@ -120,5 +121,5 @@
       <axis xyz="0 0 1"/>
       <limit lower="-${max_steer_angle}" upper="${max_steer_angle}" effort="100.0" velocity="2.0"/>
-      <dynamics damping="0.001" friction="0.05"/> <!-- Add this line -->
+      <dynamics damping="0.001" friction="0.05"/>
     </joint>
     <xacro:rc_wheel prefix="${prefix}" mesh_rpy="${mesh_rpy}"/>
@@ -129,9 +130,118 @@
       <axis xyz="0 0 1"/>
       <limit effort="5.0" velocity="100.0"/>
-      <dynamics damping="0.001" friction="0.05"/> <!-- Add this line -->
+      <dynamics damping="0.001" friction="0.05"/>
     </joint>
   </xacro:macro>
   <xacro:front_steer_assembly prefix="front_left" y_offset="${track_width/2}" mesh_rpy="-${M_PI/2.0} 0 0"/>
   <xacro:front_steer_assembly prefix="front_right" y_offset="-${track_width/2}" mesh_rpy="${M_PI/2.0} 0 0"/>
+  <!-- =============================== -->
+  <!-- INTEGRATED RPLIDAR A1           -->
+  <!-- =============================== -->
+  <material name="black_lidar">
+    <color rgba="0 0 0 1" />
+  </material>
+  <joint name="laser_joint" type="fixed">
+    <parent link="base_link"/>
+    <child link="laser_frame"/>
+    <origin xyz="0.14 0 0.1" rpy="0 0 ${M_PI}"/>
+  </joint>
+<link name="laser_frame">
+    <visual>
+      <origin xyz="0 0 -0.01" rpy="0 0 0"/>
+      <geometry>
+        <mesh filename="file://$(find rc_car_description)/meshes/rplidar_a1.STL" />
+      </geometry>
+      <material name="black_lidar"/>
+    </visual>
+    <collision>
+      <origin xyz="0 0 -0.01" rpy="0 0 0"/>
+      <geometry>
+        <!-- Replaced the STL mesh with a simple cylinder to prevent segfaults -->
+        <cylinder radius="0.035" length="0.05"/>
+      </geometry>
+    </collision>
+    <xacro:dummy_inertia/>
+  </link>
+  <gazebo reference="laser_frame">
+    <material>Gazebo/Black</material>
+    <sensor name="laser" type="ray">
+      <pose> 0 0 0 0 0 0 </pose>
+      <visualize>true</visualize>
+      <update_rate>5.5</update_rate>
+      <ray>
+        <scan>
+          <horizontal>
+            <samples>363</samples>
+            <resolution>1</resolution>
+            <min_angle>${-M_PI}</min_angle>
+            <max_angle>${M_PI}</max_angle>
+          </horizontal>
+        </scan>
+        <range>
+          <min>0.15</min>
+          <max>12.0</max>
+          <resolution>0.05</resolution>
+        </range>
+        <noise>
+          <type>gaussian</type>
+          <mean>0.0</mean>
+          <stddev>0.01</stddev>
+        </noise>
+      </ray>
+      <plugin name="laser_controller" filename="libgazebo_ros_ray_sensor.so">
+        <ros>
+          <remapping>~/out:=scan_raw</remapping>
+        </ros>
+        <output_type>sensor_msgs/LaserScan</output_type>
+        <frame_name>laser_frame</frame_name>
+      </plugin>
+    </sensor>
+  </gazebo>
+<!-- =============================== -->
+  <!-- INTEGRATED JETSON NANO          -->
+  <!-- =============================== -->
+  <material name="green_pcb">
+    <color rgba="0 0.5 0 1" />
+  </material>
+  <joint name="jetson_joint" type="fixed">
+    <parent link="base_link"/>
+    <child link="jetson_link"/>
+    <!-- Positioned behind the LiDAR. Adjust the negative X value to slide it further back if needed. -->
+    <origin xyz="-0.02 0 0.06" rpy="0 0 0"/>
+  </joint>
+<link name="jetson_link">
+    <visual>
+      <origin xyz="0 0 0" rpy="0 0 0"/>
+      <geometry>
+        <!-- Change the extension from .stl to .dae -->
+        <mesh filename="file://$(find rc_car_description)/meshes/jetson_nano.dae" scale="0.001 0.001 0.001"/>
+      </geometry>
+      <!-- The <material> tag is removed because the .dae handles it natively -->
+    </visual>
+    <xacro:dummy_inertia/>
+  </link>
+  <!-- =============================== -->
+  <!-- HC-SR04 ULTRASONIC SENSOR       -->
+  <!-- =============================== -->
+  <joint name="ultrasonic_joint" type="fixed">
+    <parent link="base_link"/>
+    <child link="ultrasonic_link"/>
+    <!-- Positioned at the front edge of the 0.25m chassis -->
+    <origin xyz="0.185 0 0.015" rpy="0 0 0"/>
+  </joint>
+  <link name="ultrasonic_link">
+    <visual>
+      <origin xyz="0 0 0" rpy="${M_PI / 2} ${M_PI} ${M_PI / 2}"/>
+      <geometry>
+        <!-- Change the extension from .stl to .dae -->
+        <mesh filename="file://$(find rc_car_description)/meshes/hc-sr-04.dae" scale="0.001 0.001 0.001"/>
+      </geometry>
+    </visual>
+    <!-- Omit collision to avoid raycast bugs -->
+    <xacro:dummy_inertia/>
+  </link>
+  <!-- =============================== -->
+  <!-- ACKERMANN DRIVE PLUGIN          -->
+  <!-- =============================== -->
   <gazebo>
     <plugin name="gazebo_ros_ackermann_drive" filename="libgazebo_ros_ackermann_drive.so">
@@ -160,7 +270,7 @@
       <robot_base_frame>base_footprint</robot_base_frame>
       <!-- PID tuning -->
-      <left_steering_pid_gain>10.0 0.0 0.1</left_steering_pid_gain>
+      <left_steering_pid_gain>50.0 0.0 0.1</left_steering_pid_gain>
       <left_steering_i_range>0 0</left_steering_i_range>
-      <right_steering_pid_gain>10.0 0.0 0.1</right_steering_pid_gain>
+      <right_steering_pid_gain>50.0 0.0 0.1</right_steering_pid_gain>
       <right_steering_i_range>0 0</right_steering_i_range>
       <linear_velocity_pid_gain>5.0 0.0 0.0</linear_velocity_pid_gain>
@@ -172,3 +282,47 @@
     </plugin>
   </gazebo>
+<gazebo reference="ultrasonic_link">
+    <material>Gazebo/Blue</material>
+    <sensor name="hcsr04" type="ray">
+      <pose>0 0 0 0 0 0</pose>
+      <!-- You can leave this true! A 5x5 ray grid won't lag your GPU like the LiDAR did -->
+      <visualize>true</visualize>
+      <update_rate>20.0</update_rate> <!-- HC-SR04 practical update rate -->
+      <ray>
+        <scan>
+          <horizontal>
+            <samples>5</samples>
+            <resolution>1</resolution>
+            <min_angle>-0.13</min_angle> <!-- -7.5 degrees -->
+            <max_angle>0.13</max_angle>  <!-- +7.5 degrees -->
+          </horizontal>
+          <vertical>
+            <samples>5</samples>
+            <resolution>1</resolution>
+            <min_angle>-0.01</min_angle>
+            <max_angle>0.0314</max_angle>
+          </vertical>
+        </scan>
+        <range>
+          <min>0.05</min> <!-- 5cm minimum range -->
+          <max>4.0</max>  <!-- 400cm maximum range -->
+          <resolution>0.01</resolution>
+        </range>
+        <noise>
+          <type>gaussian</type>
+          <mean>0.0</mean>
+          <stddev>0.025</stddev>
+        </noise>
+      </ray>
+      <plugin name="ultrasonic_sensor" filename="libgazebo_ros_ray_sensor.so">
+        <ros>
+          <remapping>~/out:=ultrasonic/range</remapping>
+        </ros>
+        <!-- Tell the plugin to format the data as a Range message, not a LaserScan -->
+        <output_type>sensor_msgs/Range</output_type>
+        <radiation_type>ultrasound</radiation_type>
+        <frame_name>ultrasonic_link</frame_name>
+      </plugin>
+    </sensor>
+  </gazebo>
 </robot>

Commit message: updated meshes

File: rc_car_description/urdf/rc_car.xacro (robot description, xacro)
@@ -2,6 +2,6 @@
 <robot xmlns:xacro="http://www.ros.org/wiki/xacro" name="rc_car">
   <xacro:property name="pkg_name" value="rc_car_description"/>
-  <xacro:property name="wheelbase" value="0.167"/>
-  <xacro:property name="chassis_x_offset" value="0.086"/>
+  <xacro:property name="wheelbase" value="0.1688"/>
+  <xacro:property name="chassis_x_offset" value="0.094"/>
   <xacro:property name="track_width" value="0.162"/>
   <xacro:property name="wheel_radius" value="0.03"/>

Commit message: rearranged car components

File: rc_car_description/urdf/rc_car.xacro (robot description, xacro)
@@ -199,4 +199,37 @@
   </gazebo>
 <!-- =============================== -->
+  <!-- LIPO BATTERY                    -->
+  <!-- =============================== -->
+  <material name="lipo_blue">
+    <color rgba="0.1 0.5 0.8 1" />
+  </material>
+  <joint name="battery_joint" type="fixed">
+    <parent link="base_link"/>
+    <child link="battery_link"/>
+    <!-- Positioned squarely between the chassis and the Jetson -->
+    <origin xyz="0.09 0 0.045" rpy="0 0 0"/>
+  </joint>
+  <link name="battery_link">
+    <visual>
+      <origin xyz="0 0 0" rpy="0 0 0"/>
+      <geometry>
+        <!-- 135mm length, 42mm width, 21mm height -->
+        <box size="0.135 0.042 0.021"/>
+      </geometry>
+      <material name="lipo_blue"/>
+    </visual>
+    <collision>
+      <origin xyz="0 0 0" rpy="0 0 0"/>
+      <geometry>
+        <box size="0.135 0.042 0.021"/>
+      </geometry>
+    </collision>
+    <!-- Adds ~250g of realistic weight to improve tire traction! -->
+    <xacro:box_inertia m="0.25" w="0.042" h="0.021" d="0.135" x_offset="0" z_offset="0"/>
+  </link>
+  <gazebo reference="battery_link">
+    <material>Gazebo/Blue</material>
+  </gazebo>
+<!-- =============================== -->
   <!-- INTEGRATED JETSON NANO          -->
   <!-- =============================== -->
@@ -208,5 +241,5 @@
     <child link="jetson_link"/>
     <!-- Positioned behind the LiDAR. Adjust the negative X value to slide it further back if needed. -->
-    <origin xyz="-0.02 0 0.06" rpy="0 0 0"/>
+    <origin xyz="-0.02 -0.02 0.06" rpy="0 0 0"/>
   </joint>
 <link name="jetson_link">
@@ -228,5 +261,5 @@
     <child link="ultrasonic_link"/>
     <!-- Positioned at the front edge of the 0.25m chassis -->
-    <origin xyz="0.185 0 0.015" rpy="0 0 0"/>
+    <origin xyz="0.19 0 0.01" rpy="0 0 0"/>
   </joint>
   <link name="ultrasonic_link">

Commit message: added map

File: rc_car_description/urdf/rc_car.xacro (robot description, xacro)
@@ -120,5 +120,5 @@
       <origin xyz="${wheelbase} ${y_offset} 0" rpy="0 0 0"/>
       <axis xyz="0 0 1"/>
-      <limit lower="-${max_steer_angle}" upper="${max_steer_angle}" effort="100.0" velocity="2.0"/>
+      <limit lower="-${max_steer_angle}" upper="${max_steer_angle}" effort="100.0" velocity="5.0"/>
       <dynamics damping="0.001" friction="0.05"/>
     </joint>
@@ -303,7 +303,7 @@
       <robot_base_frame>base_footprint</robot_base_frame>
       <!-- PID tuning -->
-      <left_steering_pid_gain>50.0 0.0 0.1</left_steering_pid_gain>
+      <left_steering_pid_gain>5.0 0.0 0.1</left_steering_pid_gain>
       <left_steering_i_range>0 0</left_steering_i_range>
-      <right_steering_pid_gain>50.0 0.0 0.1</right_steering_pid_gain>
+      <right_steering_pid_gain>5.0 0.0 0.1</right_steering_pid_gain>
       <right_steering_i_range>0 0</right_steering_i_range>
       <linear_velocity_pid_gain>5.0 0.0 0.0</linear_velocity_pid_gain>

Commit message: add slam and switched car models to lower poly ones for better performance

File: rc_car_description/urdf/rc_car.xacro (robot description, xacro)
@@ -40,5 +40,5 @@
       <origin xyz="${chassis_x_offset} 0 0" rpy="0 0 0"/>
       <geometry>
-        <mesh filename="file://$(find rc_car_description)/meshes/rc_car_chassis.stl" scale="1 1 1"/>
+        <mesh filename="file://$(find rc_car_description)/meshes/rc_car_chassis_light.stl" scale="1 1 1"/>
       </geometry>
       <material name="gray">
@@ -70,5 +70,5 @@
         <origin xyz="0 0 0" rpy="${mesh_rpy}"/>
         <geometry>
-          <mesh filename="file://$(find rc_car_description)/meshes/rc_car_wheel.stl" scale="1 1 1"/>
+          <mesh filename="file://$(find rc_car_description)/meshes/rc_car_wheel_light.stl" scale="1 1 1"/>
         </geometry>
         <material name="black">
@@ -168,9 +168,9 @@
       <pose> 0 0 0 0 0 0 </pose>
       <visualize>true</visualize>
-      <update_rate>5.5</update_rate>
+      <update_rate>10.0</update_rate>
       <ray>
         <scan>
           <horizontal>
-            <samples>363</samples>
+            <samples>360</samples>
             <resolution>1</resolution>
             <min_angle>${-M_PI}</min_angle>
@@ -186,5 +186,5 @@
           <type>gaussian</type>
           <mean>0.0</mean>
-          <stddev>0.01</stddev>
+          <stddev>0.012</stddev>
         </noise>
       </ray>
