Commit message: updated sim params

File: rc_car_description/urdf/rc_car.xacro (robot description, xacro)
@@ -1,361 +1,7 @@
 <?xml version="1.0"?>
 <robot xmlns:xacro="http://www.ros.org/wiki/xacro" name="rc_car">
-  <xacro:property name="pkg_name" value="rc_car_description"/>
-  <xacro:property name="wheelbase" value="0.1688"/>
-  <xacro:property name="chassis_x_offset" value="0.094"/>
-  <xacro:property name="track_width" value="0.162"/>
-  <xacro:property name="wheel_radius" value="0.03"/>
-  <xacro:property name="wheel_width" value="0.03"/>
-  <xacro:property name="max_steer_angle" value="0.523"/>
-  <xacro:property name="M_PI" value="3.1415926535897931" />
-  <xacro:macro name="box_inertia" params="m w h d x_offset z_offset">
-    <inertial>
-      <origin xyz="${x_offset} 0 ${z_offset}" rpy="0 0 0"/>
-      <mass value="${m}"/>
-      <inertia ixx="${(m/12) * (h*h + d*d)}" ixy="0.0" ixz="0.0" iyy="${(m/12) * (w*w + d*d)}" iyz="0.0" izz="${(m/12) * (w*w + h*h)}"/>
-    </inertial>
-  </xacro:macro>
-  <xacro:macro name="cylinder_inertia" params="m r h">
-    <inertial>
-      <origin xyz="0 0 0" rpy="0 0 0"/>
-      <mass value="${m}"/>
-      <inertia ixx="${(m/12) * (3*r*r + h*h)}" ixy="0" ixz="0" iyy="${(m/12) * (3*r*r + h*h)}" iyz="0" izz="${(m/2) * (r*r)}"/>
-    </inertial>
-  </xacro:macro>
-  <xacro:macro name="dummy_inertia">
-    <inertial>
-      <origin xyz="0 0 0" rpy="0 0 0"/>
-      <mass value="0.1"/>
-      <inertia ixx="1e-3" ixy="0" ixz="0" iyy="1e-3" iyz="0" izz="1e-3"/>
-    </inertial>
-  </xacro:macro>
-  <link name="base_footprint"/>
-  <joint name="base_footprint_joint" type="fixed">
-    <parent link="base_footprint"/>
-    <child link="base_link"/>
-    <origin xyz="0 0 ${wheel_radius}" rpy="0 0 0"/>
-  </joint>
-  <link name="base_link">
-    <visual>
-      <origin xyz="${chassis_x_offset} 0 0" rpy="0 0 0"/>
-      <geometry>
-        <mesh filename="file://$(find rc_car_description)/meshes/rc_car_chassis_light.stl" scale="1 1 1"/>
-      </geometry>
-      <material name="gray">
-        <color rgba="0.5 0.5 0.5 1.0"/>
-      </material>
-    </visual>
-    <collision>
-      <origin xyz="${chassis_x_offset} 0 0.015" rpy="0 0 0"/>
-      <geometry>
-        <box size="0.25 0.08 0.05"/>
-      </geometry>
-    </collision>
-    <xacro:box_inertia m="1.5" w="0.12" h="0.05" d="0.25" x_offset="${chassis_x_offset}" z_offset="-0.02"/>
-  </link>
-  <!-- Dummy Steering Wheel to satisfy the Ackermann plugin -->
-  <link name="steering_wheel_link">
-    <xacro:dummy_inertia/>
-  </link>
-  <joint name="steering_wheel_joint" type="revolute">
-    <parent link="base_link"/>
-    <child link="steering_wheel_link"/>
-    <origin xyz="0 0 0" rpy="0 0 0"/>
-    <axis xyz="0 0 1"/>
-    <limit lower="-${max_steer_angle}" upper="${max_steer_angle}" effort="10.0" velocity="10.0"/>
-  </joint>
-  <xacro:macro name="rc_wheel" params="prefix mesh_rpy">
-    <link name="${prefix}_wheel_link">
-      <visual>
-        <origin xyz="0 0 0" rpy="${mesh_rpy}"/>
-        <geometry>
-          <mesh filename="file://$(find rc_car_description)/meshes/rc_car_wheel_light.stl" scale="1 1 1"/>
-        </geometry>
-        <material name="black">
-          <color rgba="0.1 0.1 0.1 1.0"/>
-        </material>
-      </visual>
-      <collision>
-        <origin xyz="0 0 0" rpy="0 0 0"/>
-        <geometry>
-          <cylinder radius="${wheel_radius}" length="${wheel_width}"/>
-        </geometry>
-      </collision>
-      <xacro:cylinder_inertia m="0.5" r="${wheel_radius}" h="${wheel_width}"/>
-    </link>
-    <gazebo reference="${prefix}_wheel_link">
-      <mu1>1.2</mu1>
-      <mu2>1.2</mu2>
-      <kp>1000000.0</kp>
-      <kd>100.0</kd>
-      <minDepth>0.001</minDepth>
-      <material>Gazebo/Black</material>
-    </gazebo>
-  </xacro:macro>
-  <xacro:rc_wheel prefix="rear_left" mesh_rpy="-${M_PI/2.0} 0 0"/>
-  <joint name="rear_left_wheel_joint" type="continuous">
-    <parent link="base_link"/>
-    <child link="rear_left_wheel_link"/>
-    <origin xyz="0 ${track_width/2} 0" rpy="-${M_PI/2.0} 0 0"/>
-    <axis xyz="0 0 1"/>
-    <limit effort="5.0" velocity="100.0"/>
-    <dynamics damping="0.001" friction="0.05"/>
-  </joint>
-  <xacro:rc_wheel prefix="rear_right" mesh_rpy="${M_PI/2.0} 0 0"/>
-  <joint name="rear_right_wheel_joint" type="continuous">
-    <parent link="base_link"/>
-    <child link="rear_right_wheel_link"/>
-    <origin xyz="0 ${-track_width/2} 0" rpy="-${M_PI/2.0} 0 0"/>
-    <axis xyz="0 0 1"/>
-    <limit effort="5.0" velocity="100.0"/>
-    <dynamics damping="0.001" friction="0.05"/>
-  </joint>
-  <xacro:macro name="front_steer_assembly" params="prefix y_offset mesh_rpy">
-    <link name="${prefix}_steer_link">
-      <xacro:dummy_inertia/>
-    </link>
-    <joint name="${prefix}_steer_joint" type="revolute">
-      <parent link="base_link"/>
-      <child link="${prefix}_steer_link"/>
-      <origin xyz="${wheelbase} ${y_offset} 0" rpy="0 0 0"/>
-      <axis xyz="0 0 1"/>
-      <limit lower="-${max_steer_angle}" upper="${max_steer_angle}" effort="100.0" velocity="5.0"/>
-      <dynamics damping="0.001" friction="0.05"/>
-    </joint>
-    <xacro:rc_wheel prefix="${prefix}" mesh_rpy="${mesh_rpy}"/>
-    <joint name="${prefix}_wheel_joint" type="continuous">
-      <parent link="${prefix}_steer_link"/>
-      <child link="${prefix}_wheel_link"/>
-      <origin xyz="0 0 0" rpy="-${M_PI/2.0} 0 0"/>
-      <axis xyz="0 0 1"/>
-      <limit effort="5.0" velocity="100.0"/>
-      <dynamics damping="0.001" friction="0.05"/>
-    </joint>
-  </xacro:macro>
-  <xacro:front_steer_assembly prefix="front_left" y_offset="${track_width/2}" mesh_rpy="-${M_PI/2.0} 0 0"/>
-  <xacro:front_steer_assembly prefix="front_right" y_offset="-${track_width/2}" mesh_rpy="${M_PI/2.0} 0 0"/>
-  <!-- =============================== -->
-  <!-- INTEGRATED RPLIDAR A1           -->
-  <!-- =============================== -->
-  <material name="black_lidar">
-    <color rgba="0 0 0 1" />
-  </material>
-  <joint name="laser_joint" type="fixed">
-    <parent link="base_link"/>
-    <child link="laser_frame"/>
-    <origin xyz="0.14 0 0.1" rpy="0 0 ${M_PI}"/>
-  </joint>
-<link name="laser_frame">
-    <visual>
-      <origin xyz="0 0 -0.01" rpy="0 0 0"/>
-      <geometry>
-        <mesh filename="file://$(find rc_car_description)/meshes/rplidar_a1.STL" />
-      </geometry>
-      <material name="black_lidar"/>
-    </visual>
-    <collision>
-      <origin xyz="0 0 -0.01" rpy="0 0 0"/>
-      <geometry>
-        <!-- Replaced the STL mesh with a simple cylinder to prevent segfaults -->
-        <cylinder radius="0.035" length="0.05"/>
-      </geometry>
-    </collision>
-    <xacro:dummy_inertia/>
-  </link>
-  <gazebo reference="laser_frame">
-    <material>Gazebo/Black</material>
-    <sensor name="laser" type="ray">
-      <pose> 0 0 0 0 0 0 </pose>
-      <visualize>true</visualize>
-      <update_rate>10.0</update_rate>
-      <ray>
-        <scan>
-          <horizontal>
-            <samples>360</samples>
-            <resolution>1</resolution>
-            <min_angle>${-M_PI}</min_angle>
-            <max_angle>${M_PI}</max_angle>
-          </horizontal>
-        </scan>
-        <range>
-          <min>0.15</min>
-          <max>12.0</max>
-          <resolution>0.05</resolution>
-        </range>
-        <noise>
-          <type>gaussian</type>
-          <mean>0.0</mean>
-          <stddev>0.012</stddev>
-        </noise>
-      </ray>
-      <plugin name="laser_controller" filename="libgazebo_ros_ray_sensor.so">
-        <ros>
-          <remapping>~/out:=scan_raw</remapping>
-        </ros>
-        <output_type>sensor_msgs/LaserScan</output_type>
-        <frame_name>laser_frame</frame_name>
-      </plugin>
-    </sensor>
-  </gazebo>
-<!-- =============================== -->
-  <!-- LIPO BATTERY                    -->
-  <!-- =============================== -->
-  <material name="lipo_blue">
-    <color rgba="0.1 0.5 0.8 1" />
-  </material>
-  <joint name="battery_joint" type="fixed">
-    <parent link="base_link"/>
-    <child link="battery_link"/>
-    <!-- Positioned squarely between the chassis and the Jetson -->
-    <origin xyz="0.09 0 0.045" rpy="0 0 0"/>
-  </joint>
-  <link name="battery_link">
-    <visual>
-      <origin xyz="0 0 0" rpy="0 0 0"/>
-      <geometry>
-        <!-- 135mm length, 42mm width, 21mm height -->
-        <box size="0.135 0.042 0.021"/>
-      </geometry>
-      <material name="lipo_blue"/>
-    </visual>
-    <collision>
-      <origin xyz="0 0 0" rpy="0 0 0"/>
-      <geometry>
-        <box size="0.135 0.042 0.021"/>
-      </geometry>
-    </collision>
-    <!-- Adds ~250g of realistic weight to improve tire traction! -->
-    <xacro:box_inertia m="0.25" w="0.042" h="0.021" d="0.135" x_offset="0" z_offset="0"/>
-  </link>
-  <gazebo reference="battery_link">
-    <material>Gazebo/Blue</material>
-  </gazebo>
-<!-- =============================== -->
-  <!-- INTEGRATED JETSON NANO          -->
-  <!-- =============================== -->
-  <material name="green_pcb">
-    <color rgba="0 0.5 0 1" />
-  </material>
-  <joint name="jetson_joint" type="fixed">
-    <parent link="base_link"/>
-    <child link="jetson_link"/>
-    <!-- Positioned behind the LiDAR. Adjust the negative X value to slide it further back if needed. -->
-    <origin xyz="-0.02 -0.02 0.06" rpy="0 0 0"/>
-  </joint>
-<link name="jetson_link">
-    <visual>
-      <origin xyz="0 0 0" rpy="0 0 0"/>
-      <geometry>
-        <!-- Change the extension from .stl to .dae -->
-        <mesh filename="file://$(find rc_car_description)/meshes/jetson_nano.dae" scale="0.001 0.001 0.001"/>
-      </geometry>
-      <!-- The <material> tag is removed because the .dae handles it natively -->
-    </visual>
-    <xacro:dummy_inertia/>
-  </link>
-  <!-- =============================== -->
-  <!-- HC-SR04 ULTRASONIC SENSOR       -->
-  <!-- =============================== -->
-  <joint name="ultrasonic_joint" type="fixed">
-    <parent link="base_link"/>
-    <child link="ultrasonic_link"/>
-    <!-- Positioned at the front edge of the 0.25m chassis -->
-    <origin xyz="0.19 0 0.01" rpy="0 0 0"/>
-  </joint>
-  <link name="ultrasonic_link">
-    <visual>
-      <origin xyz="0 0 0" rpy="${M_PI / 2} ${M_PI} ${M_PI / 2}"/>
-      <geometry>
-        <!-- Change the extension from .stl to .dae -->
-        <mesh filename="file://$(find rc_car_description)/meshes/hc-sr-04.dae" scale="0.001 0.001 0.001"/>
-      </geometry>
-    </visual>
-    <!-- Omit collision to avoid raycast bugs -->
-    <xacro:dummy_inertia/>
-  </link>
-  <!-- =============================== -->
-  <!-- ACKERMANN DRIVE PLUGIN          -->
-  <!-- =============================== -->
-  <gazebo>
-    <plugin name="gazebo_ros_ackermann_drive" filename="libgazebo_ros_ackermann_drive.so">
-      <ros>
-        <namespace>/</namespace>
-        <remapping>cmd_vel:=cmd_vel</remapping>
-        <remapping>odom:=odom</remapping>
-        <remapping>distance:=distance</remapping>
-      </ros>
-      <update_rate>100.0</update_rate>
-      <front_left_joint>front_left_wheel_joint</front_left_joint>
-      <front_right_joint>front_right_wheel_joint</front_right_joint>
-      <rear_left_joint>rear_left_wheel_joint</rear_left_joint>
-      <rear_right_joint>rear_right_wheel_joint</rear_right_joint>
-      <left_steering_joint>front_left_steer_joint</left_steering_joint>
-      <right_steering_joint>front_right_steer_joint</right_steering_joint>
-      <steering_wheel_joint>steering_wheel_joint</steering_wheel_joint>
-      <wheel_separation>${track_width}</wheel_separation>
-      <wheel_base>${wheelbase}</wheel_base>
-      <steering_wheel_angle>${max_steer_angle}</steering_wheel_angle>
-      <wheel_radius>${wheel_radius}</wheel_radius>
-      <max_steer>${max_steer_angle}</max_steer>
-      <max_steering_angle>${max_steer_angle}</max_steering_angle>
-      <max_speed>5.0</max_speed>
-      <odometry_frame>odom</odometry_frame>
-      <robot_base_frame>base_footprint</robot_base_frame>
-      <!-- PID tuning -->
-      <left_steering_pid_gain>5.0 0.0 0.1</left_steering_pid_gain>
-      <left_steering_i_range>0 0</left_steering_i_range>
-      <right_steering_pid_gain>5.0 0.0 0.1</right_steering_pid_gain>
-      <right_steering_i_range>0 0</right_steering_i_range>
-      <linear_velocity_pid_gain>5.0 0.0 0.0</linear_velocity_pid_gain>
-      <linear_velocity_i_range>0 0</linear_velocity_i_range>
-      <publish_odom>true</publish_odom>
-      <publish_odom_tf>true</publish_odom_tf>
-      <publish_wheel_tf>true</publish_wheel_tf>
-      <publish_distance>true</publish_distance>
-    </plugin>
-  </gazebo>
-<gazebo reference="ultrasonic_link">
-    <material>Gazebo/Blue</material>
-    <sensor name="hcsr04" type="ray">
-      <pose>0 0 0 0 0 0</pose>
-      <!-- You can leave this true! A 5x5 ray grid won't lag your GPU like the LiDAR did -->
-      <visualize>true</visualize>
-      <update_rate>20.0</update_rate> <!-- HC-SR04 practical update rate -->
-      <ray>
-        <scan>
-          <horizontal>
-            <samples>5</samples>
-            <resolution>1</resolution>
-            <min_angle>-0.13</min_angle> <!-- -7.5 degrees -->
-            <max_angle>0.13</max_angle>  <!-- +7.5 degrees -->
-          </horizontal>
-          <vertical>
-            <samples>5</samples>
-            <resolution>1</resolution>
-            <min_angle>-0.01</min_angle>
-            <max_angle>0.0314</max_angle>
-          </vertical>
-        </scan>
-        <range>
-          <min>0.05</min> <!-- 5cm minimum range -->
-          <max>4.0</max>  <!-- 400cm maximum range -->
-          <resolution>0.01</resolution>
-        </range>
-        <noise>
-          <type>gaussian</type>
-          <mean>0.0</mean>
-          <stddev>0.025</stddev>
-        </noise>
-      </ray>
-      <plugin name="ultrasonic_sensor" filename="libgazebo_ros_ray_sensor.so">
-        <ros>
-          <remapping>~/out:=ultrasonic/range</remapping>
-        </ros>
-        <!-- Tell the plugin to format the data as a Range message, not a LaserScan -->
-        <output_type>sensor_msgs/Range</output_type>
-        <radiation_type>ultrasound</radiation_type>
-        <frame_name>ultrasonic_link</frame_name>
-      </plugin>
-    </sensor>
-  </gazebo>
+  <xacro:include filename="common_macros.xacro" />
+  <xacro:include filename="rc_car_core.xacro" />
+  <xacro:include filename="sensors.xacro" />
+  <xacro:include filename="gazebo.xacro" />
 </robot>
