Commit message: first working ros2_control version that moves very janky

File: rc_car_description/urdf/gazebo.xacro (robot description, xacro)
@@ -2,38 +2,11 @@
 <robot xmlns:xacro="http://www.ros.org/wiki/xacro">
   <gazebo>
-    <plugin name="gazebo_ros_ackermann_drive" filename="libgazebo_ros_ackermann_drive.so">
+    <plugin filename="libgazebo_ros2_control.so" name="gazebo_ros2_control">
+      <parameters>$(find rc_car_description)/config/controllers.yaml</parameters>
       <ros>
-        <namespace>/</namespace>
-        <remapping>cmd_vel:=cmd_vel</remapping>
-        <remapping>odom:=odom</remapping>
-        <remapping>distance:=distance</remapping>
+        <remapping>/ackermann_steering_controller/tf_odometry:=/tf</remapping>
+        <remapping>/ackermann_steering_controller/reference_unstamped:=/cmd_vel</remapping>
+        <remapping>/ackermann_steering_controller/odometry:=/odom</remapping>
       </ros>
-      <update_rate>100.0</update_rate>
-      <front_left_joint>front_left_wheel_joint</front_left_joint>
-      <front_right_joint>front_right_wheel_joint</front_right_joint>
-      <rear_left_joint>rear_left_wheel_joint</rear_left_joint>
-      <rear_right_joint>rear_right_wheel_joint</rear_right_joint>
-      <left_steering_joint>front_left_steer_joint</left_steering_joint>
-      <right_steering_joint>front_right_steer_joint</right_steering_joint>
-      <steering_wheel_joint>steering_wheel_joint</steering_wheel_joint>
-      <wheel_separation>${track_width}</wheel_separation>
-      <wheel_base>${wheelbase}</wheel_base>
-      <steering_wheel_angle>${max_steer_angle}</steering_wheel_angle>
-      <wheel_radius>${wheel_radius}</wheel_radius>
-      <max_steer>${max_steer_angle}</max_steer>
-      <max_steering_angle>${max_steer_angle}</max_steering_angle>
-      <max_speed>30.0</max_speed>
-      <odometry_frame>odom</odometry_frame>
-      <robot_base_frame>base_footprint</robot_base_frame>
-      <left_steering_pid_gain>8.0 0.0 0.003</left_steering_pid_gain>
-      <left_steering_i_range>0 0</left_steering_i_range>
-      <right_steering_pid_gain>8.0 0.0 0.003</right_steering_pid_gain>
-      <right_steering_i_range>0 0</right_steering_i_range>
-      <linear_velocity_pid_gain>50.0 0.0 0.0</linear_velocity_pid_gain>
-      <linear_velocity_i_range>0 0</linear_velocity_i_range>
-      <publish_odom>true</publish_odom>
-      <publish_odom_tf>true</publish_odom_tf>
-      <publish_wheel_tf>true</publish_wheel_tf>
-      <publish_distance>true</publish_distance>
     </plugin>
   </gazebo>

File: rc_car_description/urdf/rc_car.xacro (robot description, xacro)
@@ -5,3 +5,4 @@
   <xacro:include filename="sensors.xacro" />
   <xacro:include filename="gazebo.xacro" />
+  <xacro:include filename="ros2_control.xacro" />
 </robot>

File: rc_car_description/urdf/rc_car_core.xacro (robot description, xacro)
@@ -23,8 +23,9 @@
     <xacro:box_inertia m="1.5" w="0.12" h="0.05" d="0.25" x_offset="${chassis_x_offset}" z_offset="-0.06"/>
   </link>
+<!--
   <link name="steering_wheel_link">
     <xacro:dummy_inertia/>
   </link>
-  <joint name="steering_wheel_joint" type="revolute">
+<joint name="steering_wheel_joint" type="revolute">
     <parent link="base_link"/>
     <child link="steering_wheel_link"/>
@@ -33,4 +34,5 @@
     <limit lower="-${max_steer_angle}" upper="${max_steer_angle}" effort="10.0" velocity="10.0"/>
   </joint>
+-->
   <xacro:macro name="rc_wheel" params="prefix mesh_rpy">
     <link name="${prefix}_wheel_link">
