Commit message: added ackermann demo that works well

File: rc_car_description/urdf/common_macros.xacro (robot description, xacro)
@@ -13,5 +13,7 @@
       <origin xyz="${x_offset} 0 ${z_offset}" rpy="0 0 0"/>
       <mass value="${m}"/>
-      <inertia ixx="${(m/12) * (h*h + d*d)}" ixy="0.0" ixz="0.0" iyy="${(m/12) * (w*w + d*d)}" iyz="0.0" izz="${(m/12) * (w*w + h*h)}"/>
+      <inertia ixx="${(m/12) * (w*w + h*h)}" ixy="0.0" ixz="0.0"
+               iyy="${(m/12) * (d*d + h*h)}" iyz="0.0"
+               izz="${(m/12) * (d*d + w*w)}"/>
     </inertial>
   </xacro:macro>
@@ -20,5 +22,13 @@
       <origin xyz="0 0 0" rpy="0 0 0"/>
       <mass value="${m}"/>
-      <inertia ixx="${(m/12) * (3*r*r + h*h)}" ixy="0" ixz="0" iyy="${(m/12) * (3*r*r + h*h)}" iyz="0" izz="${(m/2) * (r*r)}"/>
+      <inertia ixx="${(m/12) * (3*r*r + h*h)}" ixy="0" ixz="0"
+               iyy="${(m/12) * (3*r*r + h*h)}" iyz="0"
+               izz="${(m/2) * (r*r)}"/>
+    </inertial>
+  </xacro:macro>
+  <xacro:macro name="steering_knuckle_inertia">
+    <inertial>
+      <origin xyz="0 0 0" rpy="0 0 0"/>
+      <mass value="0.015"/> <inertia ixx="1e-6" ixy="0" ixz="0" iyy="1e-6" iyz="0" izz="1e-6"/>
     </inertial>
   </xacro:macro>
@@ -26,6 +36,5 @@
     <inertial>
       <origin xyz="0 0 0" rpy="0 0 0"/>
-      <mass value="0.1"/>
-      <inertia ixx="1e-3" ixy="0" ixz="0" iyy="1e-3" iyz="0" izz="1e-3"/>
+      <mass value="0.01"/> <inertia ixx="1e-6" ixy="0" ixz="0" iyy="1e-6" iyz="0" izz="1e-6"/>
     </inertial>
   </xacro:macro>

File: rc_car_description/urdf/rc_car_core.xacro (robot description, xacro)
@@ -21,5 +21,5 @@
       </geometry>
     </collision>
-    <xacro:box_inertia m="1.5" w="0.12" h="0.05" d="0.25" x_offset="${chassis_x_offset}" z_offset="-0.06"/>
+    <xacro:box_inertia m="1.5" w="0.12" h="0.05" d="0.25" x_offset="${chassis_x_offset}" z_offset="0.015"/>
   </link>
 <!--
@@ -50,11 +50,11 @@
         </geometry>
       </collision>
-      <xacro:cylinder_inertia m="0.5" r="${wheel_radius}" h="${wheel_width}"/>
+      <xacro:cylinder_inertia m="0.05" r="${wheel_radius}" h="${wheel_width}"/>
     </link>
     <gazebo reference="${prefix}_wheel_link">
-      <mu1>1.2</mu1>
-      <mu2>1.2</mu2>
-      <kp>1000000.0</kp>
-      <kd>100.0</kd>
+      <mu1>1.0</mu1>
+      <mu2>1.0</mu2>
+      <kp>10000000.0</kp>
+      <kd>1.0</kd>
       <minDepth>0.001</minDepth>
       <material>Gazebo/Black</material>
@@ -67,6 +67,6 @@
     <origin xyz="0 ${track_width/2} 0" rpy="-${M_PI/2.0} 0 0"/>
     <axis xyz="0 0 1"/>
-    <limit effort="5.0" velocity="100.0"/>
-    <dynamics damping="0.001" friction="0.05"/>
+    <limit effort="10.0" velocity="100.0"/>
+    <dynamics damping="0.01" friction="0.05"/>
   </joint>
   <xacro:rc_wheel prefix="rear_right" mesh_rpy="${M_PI/2.0} 0 0"/>
@@ -76,6 +76,6 @@
     <origin xyz="0 ${-track_width/2} 0" rpy="-${M_PI/2.0} 0 0"/>
     <axis xyz="0 0 1"/>
-    <limit effort="5.0" velocity="100.0"/>
-    <dynamics damping="0.001" friction="0.05"/>
+    <limit effort="10.0" velocity="100.0"/>
+    <dynamics damping="0.01" friction="0.05"/>
   </joint>
   <xacro:macro name="front_steer_assembly" params="prefix y_offset mesh_rpy">
@@ -89,5 +89,5 @@
       <axis xyz="0 0 1"/>
       <limit lower="-${max_steer_angle}" upper="${max_steer_angle}" effort="100.0" velocity="2.0"/>
-      <dynamics damping="0.001" friction="0.05"/>
+      <dynamics damping="0.1" friction="0.01"/>
     </joint>
     <xacro:rc_wheel prefix="${prefix}" mesh_rpy="${mesh_rpy}"/>
@@ -98,5 +98,5 @@
       <axis xyz="0 0 1"/>
       <limit effort="5.0" velocity="100.0"/>
-      <dynamics damping="0.001" friction="0.05"/>
+      <dynamics damping="0.0" friction="0.0"/>
     </joint>
   </xacro:macro>
