Commit message: added front wheel joint transformations

File: ackermann_demo/urdf/gazebo.xacro (robot description, xacro)
@@ -12,4 +12,12 @@
     <joint name="rear_right_wheel_joint">
       <command_interface name="velocity"/>
+      <state_interface name="position"/>
+      <state_interface name="velocity"/>
+    </joint>
+    <joint name="front_left_wheel_joint">
+      <state_interface name="position"/>
+      <state_interface name="velocity"/>
+    </joint>
+    <joint name="front_right_wheel_joint">
       <state_interface name="position"/>
       <state_interface name="velocity"/>
