Commit message: working acerkmann

File: ackermann_demo/urdf/car.urdf.xacro (robot description, xacro)
@@ -6,14 +6,14 @@
   <link name="chassis">
     <visual>
-      <geometry> <box size="1.5 0.6 0.3"/> </geometry>
+      <geometry> <box size="0.22 0.08 0.05"/> </geometry>
       <material name="blue"/>
     </visual>
     <collision>
-      <geometry> <box size="1.5 0.6 0.3"/> </geometry>
+      <geometry> <box size="0.22 0.08 0.05"/> </geometry>
     </collision>
     <inertial>
-      <mass value="20.0"/>
+      <mass value="2.0"/>
       <origin xyz="0 0 0" rpy="0 0 0"/>
-      <inertia ixx="0.75" ixy="0.0" ixz="0.0" iyy="4.35" iyz="0.0" izz="4.35"/>
+      <inertia ixx="0.001483" ixy="0.0" ixz="0.0" iyy="0.008483" iyz="0.0" izz="0.009133"/>
     </inertial>
   </link>
@@ -21,5 +21,5 @@
     <parent link="base_link"/>
     <child link="chassis"/>
-    <origin xyz="0 0 0.2" rpy="0 0 0"/>
+    <origin xyz="0 0 0.05" rpy="0 0 0"/>
   </joint>
   <xacro:macro name="wheel_inertial" params="mass radius length">
@@ -34,17 +34,17 @@
     <visual>
       <origin rpy="1.5708 0 0" xyz="0 0 0"/>
-      <geometry> <cylinder radius="0.2" length="0.1"/> </geometry>
+      <geometry> <cylinder radius="0.03" length="0.03"/> </geometry>
       <material name="black"/>
     </visual>
     <collision>
       <origin rpy="1.5708 0 0" xyz="0 0 0"/>
-      <geometry> <cylinder radius="0.2" length="0.1"/> </geometry>
+      <geometry> <cylinder radius="0.03" length="0.03"/> </geometry>
     </collision>
-    <xacro:wheel_inertial mass="5.0" radius="0.2" length="0.1"/>
+    <xacro:wheel_inertial mass="0.1" radius="0.03" length="0.03"/>
   </link>
   <joint name="rear_left_wheel_joint" type="continuous">
     <parent link="chassis"/>
     <child link="rear_left_wheel"/>
-    <origin xyz="-0.5 0.35 -0.1" rpy="0 0 0"/>
+    <origin xyz="-0.08 0.055 -0.02" rpy="0 0 0"/>
     <axis xyz="0 1 0"/>
   </joint>
@@ -52,23 +52,23 @@
     <visual>
       <origin rpy="1.5708 0 0" xyz="0 0 0"/>
-      <geometry> <cylinder radius="0.2" length="0.1"/> </geometry>
+      <geometry> <cylinder radius="0.03" length="0.03"/> </geometry>
       <material name="black"/>
     </visual>
     <collision>
       <origin rpy="1.5708 0 0" xyz="0 0 0"/>
-      <geometry> <cylinder radius="0.2" length="0.1"/> </geometry>
+      <geometry> <cylinder radius="0.03" length="0.03"/> </geometry>
     </collision>
-    <xacro:wheel_inertial mass="5.0" radius="0.2" length="0.1"/>
+    <xacro:wheel_inertial mass="0.1" radius="0.03" length="0.03"/>
   </link>
   <joint name="rear_right_wheel_joint" type="continuous">
     <parent link="chassis"/>
     <child link="rear_right_wheel"/>
-    <origin xyz="-0.5 -0.35 -0.1" rpy="0 0 0"/>
+    <origin xyz="-0.08 -0.055 -0.02" rpy="0 0 0"/>
     <axis xyz="0 1 0"/>
   </joint>
   <link name="front_left_steer">
     <inertial>
-      <mass value="1.0"/>
-      <inertia ixx="0.01" ixy="0.0" ixz="0.0" iyy="0.01" iyz="0.0" izz="0.01"/>
+      <mass value="0.02"/>
+      <inertia ixx="0.0001" ixy="0.0" ixz="0.0" iyy="0.0001" iyz="0.0" izz="0.0001"/>
     </inertial>
   </link>
@@ -76,20 +76,20 @@
     <parent link="chassis"/>
     <child link="front_left_steer"/>
-    <origin xyz="0.5 0.35 -0.1" rpy="0 0 0"/>
+    <origin xyz="0.08 0.055 -0.02" rpy="0 0 0"/>
     <axis xyz="0 0 1"/>
-    <limit lower="-0.6" upper="0.6" effort="200.0" velocity="4.0"/>
-    <dynamics damping="2.0" friction="0.3"/>
+    <limit lower="-0.5236" upper="0.5236" effort="20.0" velocity="4.0"/>
+    <dynamics damping="0.1" friction="0.02"/>
   </joint>
   <link name="front_left_wheel">
     <visual>
       <origin rpy="1.5708 0 0" xyz="0 0 0"/>
-      <geometry> <cylinder radius="0.2" length="0.1"/> </geometry>
+      <geometry> <cylinder radius="0.03" length="0.03"/> </geometry>
       <material name="black"/>
     </visual>
     <collision>
       <origin rpy="1.5708 0 0" xyz="0 0 0"/>
-      <geometry> <cylinder radius="0.2" length="0.1"/> </geometry>
+      <geometry> <cylinder radius="0.03" length="0.03"/> </geometry>
     </collision>
-    <xacro:wheel_inertial mass="5.0" radius="0.2" length="0.1"/>
+    <xacro:wheel_inertial mass="0.1" radius="0.03" length="0.03"/>
   </link>
   <joint name="front_left_wheel_joint" type="continuous">
@@ -101,6 +101,6 @@
   <link name="front_right_steer">
     <inertial>
-      <mass value="1.0"/>
-      <inertia ixx="0.01" ixy="0.0" ixz="0.0" iyy="0.01" iyz="0.0" izz="0.01"/>
+      <mass value="0.02"/>
+      <inertia ixx="0.0001" ixy="0.0" ixz="0.0" iyy="0.0001" iyz="0.0" izz="0.0001"/>
     </inertial>
   </link>
@@ -108,20 +108,20 @@
     <parent link="chassis"/>
     <child link="front_right_steer"/>
-    <origin xyz="0.5 -0.35 -0.1" rpy="0 0 0"/>
+    <origin xyz="0.08 -0.055 -0.02" rpy="0 0 0"/>
     <axis xyz="0 0 1"/>
-    <limit lower="-0.6" upper="0.6" effort="200.0" velocity="4.0"/>
-    <dynamics damping="2.0" friction="0.3"/>
+    <limit lower="-0.5236" upper="0.5236" effort="20.0" velocity="4.0"/>
+    <dynamics damping="0.1" friction="0.02"/>
   </joint>
   <link name="front_right_wheel">
     <visual>
       <origin rpy="1.5708 0 0" xyz="0 0 0"/>
-      <geometry> <cylinder radius="0.2" length="0.1"/> </geometry>
+      <geometry> <cylinder radius="0.03" length="0.03"/> </geometry>
       <material name="black"/>
     </visual>
     <collision>
       <origin rpy="1.5708 0 0" xyz="0 0 0"/>
-      <geometry> <cylinder radius="0.2" length="0.1"/> </geometry>
+      <geometry> <cylinder radius="0.03" length="0.03"/> </geometry>
     </collision>
-    <xacro:wheel_inertial mass="5.0" radius="0.2" length="0.1"/>
+    <xacro:wheel_inertial mass="0.1" radius="0.03" length="0.03"/>
   </link>
   <joint name="front_right_wheel_joint" type="continuous">
@@ -173,26 +173,14 @@
   </gazebo>
   <gazebo reference="front_left_wheel">
-    <mu1>1.5</mu1>
-    <mu2>1.5</mu2>
-    <kp>1000000.0</kp>
-    <kd>100.0</kd>
+    <mu1>1.5</mu1> <mu2>1.5</mu2> <kp>1000000.0</kp> <kd>100.0</kd>
   </gazebo>
   <gazebo reference="front_right_wheel">
-    <mu1>1.5</mu1>
-    <mu2>1.5</mu2>
-    <kp>1000000.0</kp>
-    <kd>100.0</kd>
+    <mu1>1.5</mu1> <mu2>1.5</mu2> <kp>1000000.0</kp> <kd>100.0</kd>
   </gazebo>
   <gazebo reference="rear_left_wheel">
-    <mu1>1.5</mu1>
-    <mu2>1.5</mu2>
-    <kp>1000000.0</kp>
-    <kd>100.0</kd>
+    <mu1>1.5</mu1> <mu2>1.5</mu2> <kp>1000000.0</kp> <kd>100.0</kd>
   </gazebo>
   <gazebo reference="rear_right_wheel">
-    <mu1>1.5</mu1>
-    <mu2>1.5</mu2>
-    <kp>1000000.0</kp>
-    <kd>100.0</kd>
+    <mu1>1.5</mu1> <mu2>1.5</mu2> <kp>1000000.0</kp> <kd>100.0</kd>
   </gazebo>
 </robot>

Commit message: very good working example

File: ackermann_demo/urdf/car.urdf.xacro (robot description, xacro)
@@ -1,4 +1,11 @@
 <?xml version="1.0"?>
 <robot name="four_wheeled_car" xmlns:xacro="http://www.ros.org/wiki/xacro">
+  <xacro:property name="pkg_name" value="ackermann_demo"/>
+  <xacro:property name="wheelbase" value="0.1688"/>
+  <xacro:property name="track_width" value="0.162"/>
+  <xacro:property name="wheel_radius" value="0.03"/>
+  <xacro:property name="wheel_width" value="0.03"/>
+  <xacro:property name="max_steer_angle" value="0.523"/>
+  <xacro:property name="M_PI" value="3.1415926535897931" />
   <material name="blue"> <color rgba="0.1 0.1 0.8 1.0"/> </material>
   <material name="black"> <color rgba="0.0 0.0 0.0 1.0"/> </material>
@@ -6,9 +13,12 @@
   <link name="chassis">
     <visual>
-      <geometry> <box size="0.22 0.08 0.05"/> </geometry>
+      <origin xyz="0 0 -0.02" rpy="0 0 0"/>
+      <geometry>
+        <mesh filename="file://$(find ackermann_demo)/meshes/rc_car_chassis_light.stl" scale="1 1 1"/>
+      </geometry>
       <material name="blue"/>
     </visual>
     <collision>
-      <geometry> <box size="0.22 0.08 0.05"/> </geometry>
+      <geometry> <box size="0.24 0.08 0.05"/> </geometry>
     </collision>
     <inertial>
@@ -34,17 +44,19 @@
     <visual>
       <origin rpy="1.5708 0 0" xyz="0 0 0"/>
-      <geometry> <cylinder radius="0.03" length="0.03"/> </geometry>
-      <material name="black"/>
-    </visual>
-    <collision>
-      <origin rpy="1.5708 0 0" xyz="0 0 0"/>
-      <geometry> <cylinder radius="0.03" length="0.03"/> </geometry>
-    </collision>
-    <xacro:wheel_inertial mass="0.1" radius="0.03" length="0.03"/>
+      <geometry>
+       <mesh filename="file://$(find ackermann_demo)/meshes/rc_car_wheel_light.stl" scale="1 1 1"/>
+      </geometry>
+      <material name="black"/>
+    </visual>
+    <collision>
+      <origin rpy="1.5708 0 0" xyz="0 0 0"/>
+      <geometry> <cylinder radius="${wheel_radius}" length="${wheel_width}"/> </geometry>
+    </collision>
+    <xacro:wheel_inertial mass="0.1" radius="${wheel_radius}" length="${wheel_width}"/>
   </link>
   <joint name="rear_left_wheel_joint" type="continuous">
     <parent link="chassis"/>
     <child link="rear_left_wheel"/>
-    <origin xyz="-0.08 0.055 -0.02" rpy="0 0 0"/>
+    <origin xyz="-${wheelbase/2} ${track_width/2} -0.02" rpy="0 0 0"/>
     <axis xyz="0 1 0"/>
   </joint>
@@ -52,17 +64,19 @@
     <visual>
       <origin rpy="1.5708 0 0" xyz="0 0 0"/>
-      <geometry> <cylinder radius="0.03" length="0.03"/> </geometry>
-      <material name="black"/>
-    </visual>
-    <collision>
-      <origin rpy="1.5708 0 0" xyz="0 0 0"/>
-      <geometry> <cylinder radius="0.03" length="0.03"/> </geometry>
-    </collision>
-    <xacro:wheel_inertial mass="0.1" radius="0.03" length="0.03"/>
+      <geometry>
+       <mesh filename="file://$(find ackermann_demo)/meshes/rc_car_wheel_light.stl" scale="1 1 1"/>
+      </geometry>
+      <material name="black"/>
+    </visual>
+    <collision>
+      <origin rpy="1.5708 0 0" xyz="0 0 0"/>
+      <geometry> <cylinder radius="${wheel_radius}" length="${wheel_width}"/> </geometry>
+    </collision>
+    <xacro:wheel_inertial mass="0.1" radius="${wheel_radius}" length="${wheel_width}"/>
   </link>
   <joint name="rear_right_wheel_joint" type="continuous">
     <parent link="chassis"/>
     <child link="rear_right_wheel"/>
-    <origin xyz="-0.08 -0.055 -0.02" rpy="0 0 0"/>
+    <origin xyz="-${wheelbase/2} -${track_width/2} -0.02" rpy="0 0 0"/>
     <axis xyz="0 1 0"/>
   </joint>
@@ -70,5 +84,5 @@
     <inertial>
       <mass value="0.02"/>
-      <inertia ixx="0.0001" ixy="0.0" ixz="0.0" iyy="0.0001" iyz="0.0" izz="0.0001"/>
+      <inertia ixx="0.0000004" ixy="0.0" ixz="0.0" iyy="0.0000004" iyz="0.0" izz="0.0000004"/>
     </inertial>
   </link>
@@ -76,7 +90,7 @@
     <parent link="chassis"/>
     <child link="front_left_steer"/>
-    <origin xyz="0.08 0.055 -0.02" rpy="0 0 0"/>
+    <origin xyz="${wheelbase/2} ${track_width/2} -0.02" rpy="0 0 0"/>
     <axis xyz="0 0 1"/>
-    <limit lower="-0.5236" upper="0.5236" effort="20.0" velocity="4.0"/>
+    <limit lower="-${max_steer_angle}" upper="${max_steer_angle}" effort="20.0" velocity="4.0"/>
     <dynamics damping="0.1" friction="0.02"/>
   </joint>
@@ -84,12 +98,14 @@
     <visual>
       <origin rpy="1.5708 0 0" xyz="0 0 0"/>
-      <geometry> <cylinder radius="0.03" length="0.03"/> </geometry>
-      <material name="black"/>
-    </visual>
-    <collision>
-      <origin rpy="1.5708 0 0" xyz="0 0 0"/>
-      <geometry> <cylinder radius="0.03" length="0.03"/> </geometry>
-    </collision>
-    <xacro:wheel_inertial mass="0.1" radius="0.03" length="0.03"/>
+      <geometry>
+       <mesh filename="file://$(find ackermann_demo)/meshes/rc_car_wheel_light.stl" scale="1 1 1"/>
+      </geometry>
+      <material name="black"/>
+    </visual>
+    <collision>
+      <origin rpy="1.5708 0 0" xyz="0 0 0"/>
+      <geometry> <cylinder radius="${wheel_radius}" length="${wheel_width}"/> </geometry>
+    </collision>
+    <xacro:wheel_inertial mass="0.1" radius="${wheel_radius}" length="${wheel_width}"/>
   </link>
   <joint name="front_left_wheel_joint" type="continuous">
@@ -102,5 +118,5 @@
     <inertial>
       <mass value="0.02"/>
-      <inertia ixx="0.0001" ixy="0.0" ixz="0.0" iyy="0.0001" iyz="0.0" izz="0.0001"/>
+      <inertia ixx="0.0000004" ixy="0.0" ixz="0.0" iyy="0.0000004" iyz="0.0" izz="0.0000004"/>
     </inertial>
   </link>
@@ -108,7 +124,7 @@
     <parent link="chassis"/>
     <child link="front_right_steer"/>
-    <origin xyz="0.08 -0.055 -0.02" rpy="0 0 0"/>
+    <origin xyz="${wheelbase/2} -${track_width/2} -0.02" rpy="0 0 0"/>
     <axis xyz="0 0 1"/>
-    <limit lower="-0.5236" upper="0.5236" effort="20.0" velocity="4.0"/>
+    <limit lower="-${max_steer_angle}" upper="${max_steer_angle}" effort="20.0" velocity="4.0"/>
     <dynamics damping="0.1" friction="0.02"/>
   </joint>
@@ -116,12 +132,14 @@
     <visual>
       <origin rpy="1.5708 0 0" xyz="0 0 0"/>
-      <geometry> <cylinder radius="0.03" length="0.03"/> </geometry>
-      <material name="black"/>
-    </visual>
-    <collision>
-      <origin rpy="1.5708 0 0" xyz="0 0 0"/>
-      <geometry> <cylinder radius="0.03" length="0.03"/> </geometry>
-    </collision>
-    <xacro:wheel_inertial mass="0.1" radius="0.03" length="0.03"/>
+      <geometry>
+       <mesh filename="file://$(find ackermann_demo)/meshes/rc_car_wheel_light.stl" scale="1 1 1"/>
+      </geometry>
+      <material name="black"/>
+    </visual>
+    <collision>
+      <origin rpy="1.5708 0 0" xyz="0 0 0"/>
+      <geometry> <cylinder radius="${wheel_radius}" length="${wheel_width}"/> </geometry>
+    </collision>
+    <xacro:wheel_inertial mass="0.1" radius="${wheel_radius}" length="${wheel_width}"/>
   </link>
   <joint name="front_right_wheel_joint" type="continuous">

Commit message: configured sensors

File: ackermann_demo/urdf/car.urdf.xacro (robot description, xacro)
@@ -8,4 +8,7 @@
   <xacro:property name="max_steer_angle" value="0.523"/>
   <xacro:property name="M_PI" value="3.1415926535897931" />
+  <xacro:include filename="$(find ackermann_demo)/urdf/macro.xacro" />
+  <xacro:include filename="$(find ackermann_demo)/urdf/gazebo.xacro" />
+  <xacro:include filename="$(find ackermann_demo)/urdf/sensors.xacro" />
   <material name="blue"> <color rgba="0.1 0.1 0.8 1.0"/> </material>
   <material name="black"> <color rgba="0.0 0.0 0.0 1.0"/> </material>
@@ -33,26 +36,5 @@
     <origin xyz="0 0 0.05" rpy="0 0 0"/>
   </joint>
-  <xacro:macro name="wheel_inertial" params="mass radius length">
-    <inertial>
-      <mass value="${mass}"/>
-      <inertia ixx="${(1/12)*mass*(3*radius*radius + length*length)}" ixy="0.0" ixz="0.0"
-               iyy="${(1/12)*mass*(3*radius*radius + length*length)}" iyz="0.0"
-               izz="${0.5*mass*radius*radius}"/>
-    </inertial>
-  </xacro:macro>
-  <link name="rear_left_wheel">
-    <visual>
-      <origin rpy="1.5708 0 0" xyz="0 0 0"/>
-      <geometry>
-       <mesh filename="file://$(find ackermann_demo)/meshes/rc_car_wheel_light.stl" scale="1 1 1"/>
-      </geometry>
-      <material name="black"/>
-    </visual>
-    <collision>
-      <origin rpy="1.5708 0 0" xyz="0 0 0"/>
-      <geometry> <cylinder radius="${wheel_radius}" length="${wheel_width}"/> </geometry>
-    </collision>
-    <xacro:wheel_inertial mass="0.1" radius="${wheel_radius}" length="${wheel_width}"/>
-  </link>
+  <xacro:rc_wheel_link name="rear_left_wheel" radius="${wheel_radius}" length="${wheel_width}"/>
   <joint name="rear_left_wheel_joint" type="continuous">
     <parent link="chassis"/>
@@ -61,18 +43,5 @@
     <axis xyz="0 1 0"/>
   </joint>
-  <link name="rear_right_wheel">
-    <visual>
-      <origin rpy="1.5708 0 0" xyz="0 0 0"/>
-      <geometry>
-       <mesh filename="file://$(find ackermann_demo)/meshes/rc_car_wheel_light.stl" scale="1 1 1"/>
-      </geometry>
-      <material name="black"/>
-    </visual>
-    <collision>
-      <origin rpy="1.5708 0 0" xyz="0 0 0"/>
-      <geometry> <cylinder radius="${wheel_radius}" length="${wheel_width}"/> </geometry>
-    </collision>
-    <xacro:wheel_inertial mass="0.1" radius="${wheel_radius}" length="${wheel_width}"/>
-  </link>
+  <xacro:rc_wheel_link name="rear_right_wheel" radius="${wheel_radius}" length="${wheel_width}"/>
   <joint name="rear_right_wheel_joint" type="continuous">
     <parent link="chassis"/>
@@ -81,124 +50,5 @@
     <axis xyz="0 1 0"/>
   </joint>
-  <link name="front_left_steer">
-    <inertial>
-      <mass value="0.02"/>
-      <inertia ixx="0.0000004" ixy="0.0" ixz="0.0" iyy="0.0000004" iyz="0.0" izz="0.0000004"/>
-    </inertial>
-  </link>
-  <joint name="front_left_steering_joint" type="revolute">
-    <parent link="chassis"/>
-    <child link="front_left_steer"/>
-    <origin xyz="${wheelbase/2} ${track_width/2} -0.02" rpy="0 0 0"/>
-    <axis xyz="0 0 1"/>
-    <limit lower="-${max_steer_angle}" upper="${max_steer_angle}" effort="20.0" velocity="4.0"/>
-    <dynamics damping="0.1" friction="0.02"/>
-  </joint>
-  <link name="front_left_wheel">
-    <visual>
-      <origin rpy="1.5708 0 0" xyz="0 0 0"/>
-      <geometry>
-       <mesh filename="file://$(find ackermann_demo)/meshes/rc_car_wheel_light.stl" scale="1 1 1"/>
-      </geometry>
-      <material name="black"/>
-    </visual>
-    <collision>
-      <origin rpy="1.5708 0 0" xyz="0 0 0"/>
-      <geometry> <cylinder radius="${wheel_radius}" length="${wheel_width}"/> </geometry>
-    </collision>
-    <xacro:wheel_inertial mass="0.1" radius="${wheel_radius}" length="${wheel_width}"/>
-  </link>
-  <joint name="front_left_wheel_joint" type="continuous">
-    <parent link="front_left_steer"/>
-    <child link="front_left_wheel"/>
-    <origin xyz="0 0 0" rpy="0 0 0"/>
-    <axis xyz="0 1 0"/>
-  </joint>
-  <link name="front_right_steer">
-    <inertial>
-      <mass value="0.02"/>
-      <inertia ixx="0.0000004" ixy="0.0" ixz="0.0" iyy="0.0000004" iyz="0.0" izz="0.0000004"/>
-    </inertial>
-  </link>
-  <joint name="front_right_steering_joint" type="revolute">
-    <parent link="chassis"/>
-    <child link="front_right_steer"/>
-    <origin xyz="${wheelbase/2} -${track_width/2} -0.02" rpy="0 0 0"/>
-    <axis xyz="0 0 1"/>
-    <limit lower="-${max_steer_angle}" upper="${max_steer_angle}" effort="20.0" velocity="4.0"/>
-    <dynamics damping="0.1" friction="0.02"/>
-  </joint>
-  <link name="front_right_wheel">
-    <visual>
-      <origin rpy="1.5708 0 0" xyz="0 0 0"/>
-      <geometry>
-       <mesh filename="file://$(find ackermann_demo)/meshes/rc_car_wheel_light.stl" scale="1 1 1"/>
-      </geometry>
-      <material name="black"/>
-    </visual>
-    <collision>
-      <origin rpy="1.5708 0 0" xyz="0 0 0"/>
-      <geometry> <cylinder radius="${wheel_radius}" length="${wheel_width}"/> </geometry>
-    </collision>
-    <xacro:wheel_inertial mass="0.1" radius="${wheel_radius}" length="${wheel_width}"/>
-  </link>
-  <joint name="front_right_wheel_joint" type="continuous">
-    <parent link="front_right_steer"/>
-    <child link="front_right_wheel"/>
-    <origin xyz="0 0 0" rpy="0 0 0"/>
-    <axis xyz="0 1 0"/>
-  </joint>
-  <ros2_control name="GazeboSystem" type="system">
-    <hardware>
-      <plugin>gazebo_ros2_control/GazeboSystem</plugin>
-    </hardware>
-    <joint name="rear_left_wheel_joint">
-      <command_interface name="velocity"/>
-      <state_interface name="position"/>
-      <state_interface name="velocity"/>
-    </joint>
-    <joint name="rear_right_wheel_joint">
-      <command_interface name="velocity"/>
-      <state_interface name="position"/>
-      <state_interface name="velocity"/>
-    </joint>
-    <joint name="front_left_steering_joint">
-      <command_interface name="position"/>
-      <state_interface name="position"/>
-      <state_interface name="velocity"/>
-    </joint>
-    <joint name="front_right_steering_joint">
-      <command_interface name="position"/>
-      <state_interface name="position"/>
-      <state_interface name="velocity"/>
-    </joint>
-  </ros2_control>
-  <gazebo>
-    <plugin name="gazebo_ros2_control" filename="libgazebo_ros2_control.so">
-      <parameters>$(find ackermann_demo)/config/controllers.yaml</parameters>
-      <ros>
-        <remapping>/ackermann_steering_controller/tf_odometry:=/tf</remapping>
-        <remapping>/ackermann_steering_controller/reference:=/cmd_vel</remapping>
-        <remapping>/ackermann_steering_controller/odometry:=/odom</remapping>
-      </ros>
-    </plugin>
-  </gazebo>
-  <gazebo reference="front_left_steering_joint">
-    <implicitSpringDamper>true</implicitSpringDamper>
-  </gazebo>
-  <gazebo reference="front_right_steering_joint">
-    <implicitSpringDamper>true</implicitSpringDamper>
-  </gazebo>
-  <gazebo reference="front_left_wheel">
-    <mu1>1.5</mu1> <mu2>1.5</mu2> <kp>1000000.0</kp> <kd>100.0</kd>
-  </gazebo>
-  <gazebo reference="front_right_wheel">
-    <mu1>1.5</mu1> <mu2>1.5</mu2> <kp>1000000.0</kp> <kd>100.0</kd>
-  </gazebo>
-  <gazebo reference="rear_left_wheel">
-    <mu1>1.5</mu1> <mu2>1.5</mu2> <kp>1000000.0</kp> <kd>100.0</kd>
-  </gazebo>
-  <gazebo reference="rear_right_wheel">
-    <mu1>1.5</mu1> <mu2>1.5</mu2> <kp>1000000.0</kp> <kd>100.0</kd>
-  </gazebo>
+  <xacro:front_steer_assembly prefix="front_left"  y_offset="${track_width/2}" mirror="1" />
+  <xacro:front_steer_assembly prefix="front_right" y_offset="${track_width/2}" mirror="-1" />
 </robot>

Commit message: integrated slam

File: ackermann_demo/urdf/car.urdf.xacro (robot description, xacro)
@@ -13,4 +13,10 @@
   <material name="blue"> <color rgba="0.1 0.1 0.8 1.0"/> </material>
   <material name="black"> <color rgba="0.0 0.0 0.0 1.0"/> </material>
+  <link name="base_footprint"/>
+  <joint name="base_footprint_joint" type="fixed">
+    <parent link="base_footprint"/>
+    <child link="base_link"/>
+    <origin xyz="0 0 ${wheel_radius}" rpy="0 0 0"/>
+  </joint>
   <link name="base_link"/>
   <link name="chassis">
@@ -23,5 +29,5 @@
     </visual>
     <collision>
-      <geometry> <box size="0.24 0.08 0.05"/> </geometry>
+      <geometry> <box size="0.22 0.08 0.05"/> </geometry>
     </collision>
     <inertial>

File: ackermann_demo/urdf/sensors.xacro (robot description, xacro)
@@ -84,5 +84,5 @@
         </scan>
         <range>
-          <min>0.15</min>
+          <min>0.2</min>
           <max>12.0</max>
           <resolution>0.05</resolution>
@@ -106,5 +106,5 @@
     <parent link="chassis"/>
     <child link="ultrasonic_link"/>
-    <origin xyz="0.105 0 -0.01" rpy="0 0 0"/>
+    <origin xyz="0.11 0 -0.01" rpy="0 0 0"/>
   </joint>
   <link name="ultrasonic_link">
@@ -137,5 +137,5 @@
             <samples>10</samples>
             <resolution>1</resolution>
-            <min_angle>-0.01</min_angle>
+            <min_angle>-0.005</min_angle>
             <max_angle>0.0628</max_angle>
           </vertical>

Commit message: added a star path smoothing and costmap node

File: ackermann_demo/urdf/car.urdf.xacro (robot description, xacro)
@@ -5,5 +5,5 @@
   <xacro:property name="track_width" value="0.162"/>
   <xacro:property name="wheel_radius" value="0.03"/>
-  <xacro:property name="wheel_width" value="0.03"/>
+  <xacro:property name="wheel_width" value="0.0275"/>
   <xacro:property name="max_steer_angle" value="0.523"/>
   <xacro:property name="M_PI" value="3.1415926535897931" />
