Commit message: Updated rc car model with new printed parts

File: ackermann_demo/urdf/car.urdf.xacro (robot description, xacro)
@@ -13,4 +13,5 @@
   <material name="blue"> <color rgba="0.1 0.1 0.8 1.0"/> </material>
   <material name="black"> <color rgba="0.0 0.0 0.0 1.0"/> </material>
+  <material name="dark_grey"> <color rgba="0.2 0.2 0.2 1.0"/> </material>
   <link name="base_footprint"/>
   <joint name="base_footprint_joint" type="fixed">
@@ -42,4 +43,70 @@
     <origin xyz="0 0 0.05" rpy="0 0 0"/>
   </joint>
+  <link name="adapter_floor">
+    <visual>
+      <origin xyz="0.09 -0.043 0" rpy="${M_PI/2} 0 ${M_PI}"/>
+      <geometry>
+        <mesh filename="file://$(find ackermann_demo)/meshes/adapter_floor.STL" scale="0.001 0.001 0.001"/>
+      </geometry>
+      <material name="dark_grey"/>
+    </visual>
+    <collision>
+      <geometry> <box size="0.16 0.07 0.005"/> </geometry>
+    </collision>
+    <inertial>
+      <mass value="0.05"/>
+      <origin xyz="0 0 0" rpy="0 0 0"/>
+      <inertia ixx="0.00002" ixy="0.0" ixz="0.0" iyy="0.0001" iyz="0.0" izz="0.0001"/>
+    </inertial>
+  </link>
+  <joint name="adapter_floor_joint" type="fixed">
+    <parent link="chassis"/>
+    <child link="adapter_floor"/>
+    <origin xyz="0.0 0.0 0.015" rpy="0 0 0"/>
+  </joint>
+  <link name="adapter_roof">
+    <visual>
+      <origin xyz="0.105 -0.05 0" rpy="${M_PI/2} 0 ${M_PI}"/>
+      <geometry>
+        <mesh filename="file://$(find ackermann_demo)/meshes/adapter_roof.STL" scale="0.001 0.001 0.001"/>
+      </geometry>
+      <material name="dark_grey"/>
+    </visual>
+    <collision>
+      <geometry> <box size="0.16 0.07 0.005"/> </geometry>
+    </collision>
+    <inertial>
+      <mass value="0.05"/>
+      <origin xyz="0 0 0" rpy="0 0 0"/>
+      <inertia ixx="0.00002" ixy="0.0" ixz="0.0" iyy="0.0001" iyz="0.0" izz="0.0001"/>
+    </inertial>
+  </link>
+  <joint name="adapter_roof_joint" type="fixed">
+    <parent link="adapter_floor"/>
+    <child link="adapter_roof"/>
+    <origin xyz="0 0 0.035" rpy="0 0 0"/>
+  </joint>
+  <link name="lidar_holder">
+    <visual>
+      <origin xyz="0.068 -0.0365 0.015" rpy="0 ${M_PI} 0"/>
+      <geometry>
+        <mesh filename="file://$(find ackermann_demo)/meshes/lidar_holder.STL" scale="0.001 0.001 0.001"/>
+      </geometry>
+      <material name="black"/>
+    </visual>
+    <collision>
+      <geometry> <cylinder radius="0.04" length="0.015"/> </geometry>
+    </collision>
+    <inertial>
+      <mass value="0.03"/>
+      <origin xyz="0 0 0" rpy="0 0 0"/>
+      <inertia ixx="0.00001" ixy="0.0" ixz="0.0" iyy="0.00001" iyz="0.0" izz="0.00002"/>
+    </inertial>
+  </link>
+  <joint name="lidar_holder_joint" type="fixed">
+    <parent link="adapter_roof"/>
+    <child link="lidar_holder"/>
+    <origin xyz="0.03 0 0.005" rpy="0 0 0"/>
+  </joint>
   <xacro:rc_wheel_link name="rear_left_wheel" radius="${wheel_radius}" length="${wheel_width}"/>
   <joint name="rear_left_wheel_joint" type="continuous">

File: ackermann_demo/urdf/sensors.xacro (robot description, xacro)
@@ -7,10 +7,10 @@
     <parent link="chassis"/>
     <child link="battery_link"/>
-    <origin xyz="0 0 0.02" rpy="0 0 0"/>
+    <origin xyz="0 0 0.032" rpy="0 0 0"/>
   </joint>
   <link name="battery_link">
     <visual>
       <origin xyz="0 0 0" rpy="0 0 0"/>
-      <geometry> <box size="0.135 0.042 0.021"/> </geometry>
+      <geometry> <box size="0.14 0.0435 0.021"/> </geometry>
       <material name="lipo_blue"/>
     </visual>
@@ -33,5 +33,5 @@
     <parent link="chassis"/>
     <child link="jetson_link"/>
-    <origin xyz="-0.11 -0.04 0.04" rpy="0 0 0"/>
+    <origin xyz="-0.1 -0.025 0.06" rpy="0 0 0"/>
   </joint>
   <link name="jetson_link">
@@ -39,5 +39,5 @@
       <origin xyz="0 0 0" rpy="0 0 0"/>
       <geometry>
-        <mesh filename="file://$(find ackermann_demo)/meshes/jetson_nano.dae" scale="0.001 0.001 0.001"/>
+        <mesh filename="file://$(find ackermann_demo)/meshes/jetson_orin_nano.dae" scale="0.001 0.001 0.001"/>
       </geometry>
     </visual>
@@ -50,5 +50,5 @@
     <parent link="chassis"/>
     <child link="laser_frame"/>
-    <origin xyz="0.06 0 0.075" rpy="0 0 ${M_PI}"/>
+    <origin xyz="0.062 0 0.096" rpy="0 0 ${M_PI}"/>
   </joint>
   <link name="laser_frame">
@@ -166,5 +166,5 @@
     <parent link="chassis"/>
     <child link="camera_link"/>
-    <origin xyz="0.1 0 0.03" rpy="0 0 0"/>
+    <origin xyz="0.086 0 0.033" rpy="0 0 0"/>
   </joint>
   <link name="camera_link">

Commit message: fixed floating base_footprint and wheel mesh orientations

File: ackermann_demo/urdf/car.urdf.xacro (robot description, xacro)
@@ -41,5 +41,5 @@
     <parent link="base_link"/>
     <child link="chassis"/>
-    <origin xyz="0 0 0.05" rpy="0 0 0"/>
+    <origin xyz="0 0 0.02" rpy="0 0 0"/>
   </joint>
   <link name="adapter_floor">
@@ -113,6 +113,6 @@
     <parent link="chassis"/>
     <child link="rear_left_wheel"/>
-    <origin xyz="-${wheelbase/2} ${track_width/2} -0.02" rpy="0 0 0"/>
-    <axis xyz="0 1 0"/>
+    <origin xyz="-${wheelbase/2} ${track_width/2} -0.02" rpy="0 0 ${M_PI}"/>
+    <axis xyz="0 -1 0"/>
   </joint>
   <xacro:rc_wheel_link name="rear_right_wheel" radius="${wheel_radius}" length="${wheel_width}"/>
@@ -125,3 +125,7 @@
   <xacro:front_steer_assembly prefix="front_left"  y_offset="${track_width/2}" mirror="1" />
   <xacro:front_steer_assembly prefix="front_right" y_offset="${track_width/2}" mirror="-1" />
+  <gazebo reference="rear_left_wheel">  <material>Gazebo/Black</material> </gazebo>
+  <gazebo reference="rear_right_wheel"> <material>Gazebo/Black</material> </gazebo>
+  <gazebo reference="front_left_wheel">  <material>Gazebo/Black</material> </gazebo>
+  <gazebo reference="front_right_wheel"> <material>Gazebo/Black</material> </gazebo>
 </robot>

File: ackermann_demo/urdf/macro.xacro (robot description, xacro)
@@ -44,6 +44,12 @@
       <parent link="${prefix}_steer"/>
       <child link="${prefix}_wheel"/>
-      <origin xyz="0 0 0" rpy="0 0 0"/>
-      <axis xyz="0 1 0"/>
+      <xacro:if value="${mirror == 1}">
+        <origin xyz="0 0 0" rpy="0 0 ${M_PI}"/>
+        <axis xyz="0 -1 0"/>
+      </xacro:if>
+      <xacro:if value="${mirror == -1}">
+        <origin xyz="0 0 0" rpy="0 0 0"/>
+        <axis xyz="0 1 0"/>
+      </xacro:if>
     </joint>
   </xacro:macro>

Commit message: very well working autonomous path following

File: ackermann_demo/urdf/car.urdf.xacro (robot description, xacro)
@@ -107,5 +107,5 @@
     <parent link="adapter_roof"/>
     <child link="lidar_holder"/>
-    <origin xyz="0.03 0 0.005" rpy="0 0 0"/>
+    <origin xyz="0.035 0 0.005" rpy="0 0 0"/>
   </joint>
   <xacro:rc_wheel_link name="rear_left_wheel" radius="${wheel_radius}" length="${wheel_width}"/>

File: ackermann_demo/urdf/gazebo.xacro (robot description, xacro)
@@ -1,7 +1,15 @@
 <?xml version="1.0"?>
 <robot xmlns:xacro="http://www.ros.org/wiki/xacro">
+  <xacro:arg name="sim_mode" default="true"/>
   <ros2_control name="GazeboSystem" type="system">
     <hardware>
-      <plugin>gazebo_ros2_control/GazeboSystem</plugin>
+      <xacro:if value="$(arg sim_mode)">
+        <plugin>gazebo_ros2_control/GazeboSystem</plugin>
+      </xacro:if>
+      <xacro:unless value="$(arg sim_mode)">
+        <plugin>ackermann_demo/AckermannHardwareInterface</plugin>
+        <param name="serial_port">/dev/ttyACM0</param>
+        <param name="baud_rate">115200</param>
+      </xacro:unless>
     </hardware>
     <joint name="rear_left_wheel_joint">

File: ackermann_demo/urdf/sensors.xacro (robot description, xacro)
@@ -4,4 +4,50 @@
   <material name="black_lidar"> <color rgba="0.1 0.1 0.1 1.0"/> </material>
   <material name="raspberry_green"> <color rgba="0.0 0.4 0.0 1.0"/> </material>
+  <link name="imu_link">
+    <visual>
+      <origin xyz="0 0 0" rpy="0 0 0"/>
+      <geometry>
+        <box size="0.015 0.015 0.005"/>
+      </geometry>
+      <material name="black"/>
+    </visual>
+    <inertial>
+      <mass value="0.005"/>
+      <origin xyz="0 0 0" rpy="0 0 0"/>
+      <inertia ixx="0.000001" ixy="0.0" ixz="0.0" iyy="0.000001" iyz="0.0" izz="0.000001"/>
+    </inertial>
+  </link>
+  <gazebo reference="imu_link">
+    <sensor name="imu_sensor" type="imu">
+      <always_on>true</always_on>
+      <update_rate>100.0</update_rate>
+      <visualize>true</visualize>
+      <topic>__default_topic__</topic>
+      <plugin name="ackermann_imu_plugin" filename="libgazebo_ros_imu_sensor.so">
+        <ros>
+          <remapping>~/out:=/imu</remapping>
+        </ros>
+        <frame_name>imu_link</frame_name>
+        <initial_orientation_as_reference>false</initial_orientation_as_reference>
+      </plugin>
+      <imu>
+        <angular_velocity>
+          <x><type>gaussian</type><mean>0.0</mean><stddev>2e-4</stddev></x>
+          <y><type>gaussian</type><mean>0.0</mean><stddev>2e-4</stddev></y>
+          <z><type>gaussian</type><mean>0.0</mean><stddev>2e-4</stddev></z>
+        </angular_velocity>
+        <linear_acceleration>
+          <x><type>gaussian</type><mean>0.0</mean><stddev>1.7e-2</stddev></x>
+          <y><type>gaussian</type><mean>0.0</mean><stddev>1.7e-2</stddev></y>
+          <z><type>gaussian</type><mean>0.0</mean><stddev>1.7e-2</stddev></z>
+        </linear_acceleration>
+      </imu>
+    </sensor>
+  </gazebo>
+  <joint name="imu_joint" type="fixed">
+    <parent link="chassis"/>
+    <child link="imu_link"/>
+    <origin xyz="0.0 0.0 0.01" rpy="0 0 0"/>
+  </joint>
   <joint name="battery_joint" type="fixed">
     <parent link="chassis"/>
@@ -50,5 +96,5 @@
     <parent link="chassis"/>
     <child link="laser_frame"/>
-    <origin xyz="0.062 0 0.096" rpy="0 0 ${M_PI}"/>
+    <origin xyz="0.068 0 0.096" rpy="0 0 ${M_PI}"/>
   </joint>
   <link name="laser_frame">
